File: OpenBMS/OSBMS Balancer Rev1.sch (KiCad schematic (older format))
At the start: 68 parts, among them P1 CONN_01X07, P2 EXT-TMP, P3 CONN_01X09, P4 CONN_01X09, Q1 BSS138, Q2 BSS138, Q3 BSS138, Q4 BSS138, Q5 BSS138, Q6 BSS138, U1 ATA6870N_BMS

Commit message: rdy for review, added req'ed bits for top board
Parts:
- D1, D2, D3, D4, D5, D6: symbol LED -> LED-RESCUE-OSBMS_Balancer_Rev1
- R1, R10, R11, R12, R13, R2, R20, R21, R22, R23, R24, R25, R26, R27, R28, R29, R3, R30, R31, R32, R33, R34, R35, R36, R37, R38, R39, R4, R40, R41, R42, R5, R6, R7, R8, R9: symbol R -> R-RESCUE-OSBMS_Balancer_Rev1
Changed lines of the file:
@@
 EESchema Schematic File Version 2
+LIBS:OSBMS Balancer Rev1-rescue
 LIBS:power
 LIBS:device
@@
 LIBS:memory
 LIBS:xilinx
-LIBS:special
 LIBS:microcontrollers
 LIBS:dsp
@@
 $EndComp
 $Comp
-L LED D1
+L LED-RESCUE-OSBMS_Balancer_Rev1 D1
 U 1 1 54154E07
 P 2300 1500
@@
 $EndComp
 $Comp
-L R R20
+L R-RESCUE-OSBMS_Balancer_Rev1 R20
 U 1 1 54154E54
 P 2700 1700
@@
 $EndComp
 $Comp
-L GND #PWR02
+L GND-RESCUE-OSBMS_Balancer_Rev1 #PWR02
 U 1 1 54188E78
 P 7750 5650
@@
 $EndComp
 $Comp
-L R R12
+L R-RESCUE-OSBMS_Balancer_Rev1 R12
 U 1 1 541899DD
 P 2950 1500
@@
 To Battery
 $Comp
-L GND #PWR03
+L GND-RESCUE-OSBMS_Balancer_Rev1 #PWR03
 U 1 1 54237CBF
 P 5400 7500
@@
 $EndComp
 $Comp
-L LED D2
+L LED-RESCUE-OSBMS_Balancer_Rev1 D2
 U 1 1 542382C4
 P 2300 2550
@@
 $EndComp
 $Comp
-L R R11
+L R-RESCUE-OSBMS_Balancer_Rev1 R11
 U 1 1 542382D0
 P 2950 2550
@@
 $EndComp
 $Comp
-L LED D3
+L LED-RESCUE-OSBMS_Balancer_Rev1 D3
 U 1 1 54238784
 P 2300 3600
@@
 $EndComp
 $Comp
-L R R10
+L R-RESCUE-OSBMS_Balancer_Rev1 R10
 U 1 1 54238790
 P 2950 3600
@@
 $EndComp
 $Comp
-L LED D6
+L LED-RESCUE-OSBMS_Balancer_Rev1 D6
 U 1 1 54238D7D
 P 2300 6750
@@
 $EndComp
 $Comp
-L R R7
+L R-RESCUE-OSBMS_Balancer_Rev1 R7
 U 1 1 54238D89
 P 2950 6750
@@
 $EndComp
 $Comp
-L LED D4
+L LED-RESCUE-OSBMS_Balancer_Rev1 D4
 U 1 1 5423904D
 P 2300 4650
@@
 $EndComp
 $Comp
-L R R9
+L R-RESCUE-OSBMS_Balancer_Rev1 R9
 U 1 1 54239059
 P 2950 4650
@@
 $EndComp
 $Comp
-L LED D5
+L LED-RESCUE-OSBMS_Balancer_Rev1 D5
 U 1 1 542395D9
 P 2300 5700
@@
 $EndComp
 $Comp
-L R R8
+L R-RESCUE-OSBMS_Balancer_Rev1 R8
 U 1 1 542395E5
 P 2950 5700
@@
 $EndComp
 $Comp
-L R R5
+L R-RESCUE-OSBMS_Balancer_Rev1 R5
 U 1 1 54244F8C
 P 5050 1250
@@
 $EndComp
 $Comp
-L R R1
+L R-RESCUE-OSBMS_Balancer_Rev1 R1
 U 1 1 5424DD8C
 P 6750 5050
@@
 $EndComp
 $Comp
-L R R3
+L R-RESCUE-OSBMS_Balancer_Rev1 R3
 U 1 1 542607A6
 P 6050 4000
@@
 $EndComp
 $Comp
-L R R2
+L R-RESCUE-OSBMS_Balancer_Rev1 R2
 U 1 1 5426080C
 P 6300 4000
@@
 $EndComp
 $Comp
-L GND #PWR04
+L GND-RESCUE-OSBMS_Balancer_Rev1 #PWR04
 U 1 1 54268087
 P 6300 1800
@@
 $EndComp
 $Comp
-L GND #PWR05
+L GND-RESCUE-OSBMS_Balancer_Rev1 #PWR05
 U 1 1 54255D02
 P 10550 4950
@@
 $EndComp
 $Comp
-L GND #PWR07
+L GND-RESCUE-OSBMS_Balancer_Rev1 #PWR07
 U 1 1 5425E157
 P 8750 5500
@@
 $EndComp
 $Comp
-L +3.3V #PWR08
+L +3.3V-RESCUE-OSBMS_Balancer_Rev1 #PWR08
 U 1 1 54266B58
 P 10550 4250
@@
 $EndComp
 $Comp
-L R R4
+L R-RESCUE-OSBMS_Balancer_Rev1 R4
 U 1 1 5426CD58
 P 5050 7300
@@
 To higher board / terminator
 $Comp
-L R R21
+L R-RESCUE-OSBMS_Balancer_Rev1 R21
 U 1 1 5437B3D2
 P 2700 1850
@@
 $EndComp
 $Comp
-L R R22
+L R-RESCUE-OSBMS_Balancer_Rev1 R22
 U 1 1 5437B41D
 P 2700 2000
@@
 $EndComp
 $Comp
-L R R23
+L R-RESCUE-OSBMS_Balancer_Rev1 R23
 U 1 1 5437B46D
 P 2700 2150
@@
 $EndComp
 $Comp
-L R R24
+L R-RESCUE-OSBMS_Balancer_Rev1 R24
 U 1 1 5437F684
 P 2700 2750
@@
 $EndComp
 $Comp
-L R R25
+L R-RESCUE-OSBMS_Balancer_Rev1 R25
 U 1 1 5437F68E
 P 2700 2900
@@
 $EndComp
 $Comp
-L R R26
+L R-RESCUE-OSBMS_Balancer_Rev1 R26
 U 1 1 5437F694
 P 2700 3050
@@
 $EndComp
 $Comp
-L R R27
+L R-RESCUE-OSBMS_Balancer_Rev1 R27
 U 1 1 5437F69A
 P 2700 3200
@@
 $EndComp
 $Comp
-L R R28
+L R-RESCUE-OSBMS_Balancer_Rev1 R28
 U 1 1 543871C9
 P 2700 3800
@@
 $EndComp
 $Comp
-L R R29
+L R-RESCUE-OSBMS_Balancer_Rev1 R29
 U 1 1 543871D1
 P 2700 3950
@@
 $EndComp
 $Comp
-L R R30
+L R-RESCUE-OSBMS_Balancer_Rev1 R30
 U 1 1 543871D7
 P 2700 4100
@@
 $EndComp
 $Comp
-L R R31
+L R-RESCUE-OSBMS_Balancer_Rev1 R31
 U 1 1 543871DD
 P 2700 4250
@@
 $EndComp
 $Comp
-L R R32
+L R-RESCUE-OSBMS_Balancer_Rev1 R32
 U 1 1 5438A579
 P 2700 4850
@@
 $EndComp
 $Comp
-L R R33
+L R-RESCUE-OSBMS_Balancer_Rev1 R33
 U 1 1 5438A581
 P 2700 5000
@@
 $EndComp
 $Comp
-L R R13
+L R-RESCUE-OSBMS_Balancer_Rev1 R13
 U 1 1 5438A587
 P 2700 5150
@@
 $EndComp
 $Comp
-L R R34
+L R-RESCUE-OSBMS_Balancer_Rev1 R34
 U 1 1 5438A58D
 P 2700 5300
@@
 $EndComp
 $Comp
-L R R35
+L R-RESCUE-OSBMS_Balancer_Rev1 R35
 U 1 1 5438AD39
 P 2700 5900
@@
 $EndComp
 $Comp
-L R R36
+L R-RESCUE-OSBMS_Balancer_Rev1 R36
 U 1 1 5438AD41
 P 2700 6050
@@
 $EndComp
 $Comp
-L R R37
+L R-RESCUE-OSBMS_Balancer_Rev1 R37
 U 1 1 5438AD47
 P 2700 6200
@@
 $EndComp
 $Comp
-L R R38
+L R-RESCUE-OSBMS_Balancer_Rev1 R38
 U 1 1 5438AD4D
 P 2700 6350
@@
 $EndComp
 $Comp
-L R R39
+L R-RESCUE-OSBMS_Balancer_Rev1 R39
 U 1 1 5438FCBF
 P 2700 6950
@@
 $EndComp
 $Comp
-L R R40
+L R-RESCUE-OSBMS_Balancer_Rev1 R40
 U 1 1 5438FCC7
 P 2700 7100
@@
 $EndComp
 $Comp
-L R R41
+L R-RESCUE-OSBMS_Balancer_Rev1 R41
 U 1 1 5438FCCD
 P 2700 7250
@@
 $EndComp
 $Comp
-L R R42
+L R-RESCUE-OSBMS_Balancer_Rev1 R42
 U 1 1 5438FCD3
 P 2700 7400
@@
 	5400 7100 5300 7100
 $Comp
-L R R6
+L R-RESCUE-OSBMS_Balancer_Rev1 R6
 U 1 1 543E273A
 P 5050 7100
